File: EN715_ExpansionBoard_ver1_2.brd (EAGLE design)
At the start: 87 x 50 mm, 50 parts, among them IC1 FE1.1S, M2 SPARKFUN_SEN-15335

Commit message: Add information for production
Parts:
- renumbered M2 to M1
Changed lines of the file:
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@@
 <drawing>
 <settings>
-<setting alwaysvectorfont="yes"/>
+<setting alwaysvectorfont="no"/>
 <setting verticaltext="up"/>
 </settings>
@@
 <attribute name="VALUE" x="-30.575" y="-22.59" size="1.27" layer="28" rot="MR90"/>
 </element>
-<element name="M2" library="SparkFun SEN-15335" package="SPARKFUN_SEN-15335" value="SPARKFUN_SEN-15335" x="-20.066" y="-7.112" smashed="yes" rot="MR0">
+<element name="M1" library="SparkFun SEN-15335" package="SPARKFUN_SEN-15335" value="SPARKFUN_SEN-15335" x="-20.066" y="-7.112" smashed="yes" rot="MR0">
 <attribute name="NAME" x="-20.066" y="4.953" size="1" layer="22" ratio="10" rot="MR0" align="center"/>
 </element>
@@
 <contactref element="USB5" pad="4"/>
 <contactref element="FL5" pad="2"/>
-<contactref element="M2" pad="GND1"/>
-<contactref element="M2" pad="GND2"/>
+<contactref element="M1" pad="GND1"/>
+<contactref element="M1" pad="GND2"/>
 <wire x1="-24.98" y1="-13.97" x2="-26.035" y2="-16.93" width="0" layer="19" extent="16-16"/>
 <wire x1="-24.98" y1="-12.065" x2="-24.98" y2="-13.97" width="0" layer="19" extent="16-16"/>
@@
 <contactref element="CH1" pad="2"/>
 <contactref element="JP8" pad="2"/>
-<contactref element="M2" pad="VIN"/>
-<contactref element="M2" pad="VIN1"/>
+<contactref element="M1" pad="VIN"/>
+<contactref element="M1" pad="VIN1"/>
 <wire x1="32.385" y1="-13.6525" x2="32.385" y2="-6.0325" width="0.381" layer="16"/>
 <wire x1="36.195" y1="-17.4625" x2="32.385" y2="-13.6525" width="0.381" layer="16"/>
@@
 <signal name="MPU9250_CS" class="1">
 <contactref element="JP8" pad="1"/>
-<contactref element="M2" pad="CS"/>
+<contactref element="M1" pad="CS"/>
 <contactref element="JP7" pad="1"/>
 <wire x1="34.3154" y1="-6.0325" x2="33.3375" y2="-6.0325" width="0.254" layer="16"/>
@@
 </signal>
 <signal name="IMU_SCL/SCLK" class="1">
-<contactref element="M2" pad="SCL/SCLK"/>
+<contactref element="M1" pad="SCL/SCLK"/>
 <contactref element="JP1" pad="1"/>
 <contactref element="JP2" pad="1"/>
@@
 <signal name="IMU_SDA/SDI" class="1">
 <contactref element="JP3" pad="1"/>
-<contactref element="M2" pad="SDA/SDI"/>
+<contactref element="M1" pad="SDA/SDI"/>
 <contactref element="JP4" pad="1"/>
 <wire x1="34.29" y1="-1.5875" x2="33.3375" y2="-1.5875" width="0.254" layer="16"/>
@@
 </signal>
 <signal name="IMU_AD0/SD0" class="1">
-<contactref element="M2" pad="AD0/SD0"/>
+<contactref element="M1" pad="AD0/SD0"/>
 <contactref element="JP5" pad="1"/>
 <contactref element="JP6" pad="1"/>
